File: STS1_EEE.kicad_sch (KiCad schematic)
At the start: 20 parts, among them J1 2477, J2 Conn_02x20_Odd_Even, J3 Conn_02x20_Odd_Even, SW1 SW_SPST, U1 coordinate_system, U10 ST_Logo

Commit message: Label RasPi Zero W pin header
Parts:
- removed D?: LED, LED_SMD:LED_0805_2012Metric, symbol Device:LED
- removed J1: 2477, 2477, symbol STS1_EEE_lib:2477
- removed J2, J3: Conn_02x20_Odd_Even, symbol Connector_Generic:Conn_02x20_Odd_Even
- removed R?: 220, Resistor_SMD:R_0603_1608Metric, symbol Device:R
- removed SW1: SW_SPST, symbol Switch:SW_SPST
Connections:
- no-connect marks 26 -> 0
Other:
- note removed: "Pi HAT"
- note removed: "Pi Zero"

Commit message: Add 3V3 LDO: could be used to set EPS_BAT_GOOD high
Parts:
- renumbered FID5 to FID2, FID2 to FID3, FID6 to FID4, FID3 to FID5, FID7 to FID6, FID4 to FID7, U10 to U2
Changed lines of the file:
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@@
 		(in_pos_files yes)
 		(dnp no)
-		(property "Reference" "FID2"
+		(property "Reference" "FID3"
 			(at 35.179 14.0716 0)
 			(show_name no)
@@
 			(project "STS1_EEE"
 				(path "/81e05c2b-9a2c-430f-84ee-6a59968cd49a"
-					(reference "FID2")
+					(reference "FID3")
 					(unit 1)
 				)
@@
 		(in_pos_files yes)
 		(dnp no)
-		(property "Reference" "FID3"
+		(property "Reference" "FID5"
 			(at 50.419 14.0716 0)
 			(show_name no)
@@
 			(project "STS1_EEE"
 				(path "/81e05c2b-9a2c-430f-84ee-6a59968cd49a"
-					(reference "FID3")
+					(reference "FID5")
 					(unit 1)
 				)
@@
 		(in_pos_files yes)
 		(dnp no)
-		(property "Reference" "FID4"
+		(property "Reference" "FID7"
 			(at 64.389 14.0716 0)
 			(show_name no)
@@
 			(project "STS1_EEE"
 				(path "/81e05c2b-9a2c-430f-84ee-6a59968cd49a"
-					(reference "FID4")
+					(reference "FID7")
 					(unit 1)
 				)
@@
 		(in_pos_files yes)
 		(dnp no)
-		(property "Reference" "#PWR0101"
+		(property "Reference" "#PWR04"
 			(at 87.63 36.83 0)
 			(hide yes)
@@
 			(project "STS1_EEE"
 				(path "/81e05c2b-9a2c-430f-84ee-6a59968cd49a"
-					(reference "#PWR0101")
+					(reference "#PWR04")
 					(unit 1)
 				)
@@
 		(in_pos_files yes)
 		(dnp no)
-		(property "Reference" "#PWR0102"
+		(property "Reference" "#PWR03"
 			(at 64.77 36.83 0)
 			(hide yes)
@@
 			(project "STS1_EEE"
 				(path "/81e05c2b-9a2c-430f-84ee-6a59968cd49a"
-					(reference "#PWR0102")
+					(reference "#PWR03")
 					(unit 1)
 				)
@@
 		(in_pos_files yes)
 		(dnp no)
-		(property "Reference" "#PWR0103"
+		(property "Reference" "#PWR02"
 			(at 40.64 36.83 0)
 			(hide yes)
@@
 			(project "STS1_EEE"
 				(path "/81e05c2b-9a2c-430f-84ee-6a59968cd49a"
-					(reference "#PWR0103")
+					(reference "#PWR02")
 					(unit 1)
 				)
@@
 		(in_pos_files yes)
 		(dnp no)
-		(property "Reference" "#PWR0104"
+		(property "Reference" "#PWR01"
 			(at 17.78 36.83 0)
 			(hide yes)
@@
 			(project "STS1_EEE"
 				(path "/81e05c2b-9a2c-430f-84ee-6a59968cd49a"
-					(reference "#PWR0104")
+					(reference "#PWR01")
 					(unit 1)
 				)
@@
 		(in_pos_files yes)
 		(dnp no)
-		(property "Reference" "FID5"
+		(property "Reference" "FID2"
 			(at 19.939 19.1516 0)
 			(show_name no)
@@
 			(project "STS1_EEE"
 				(path "/81e05c2b-9a2c-430f-84ee-6a59968cd49a"
-					(reference "FID5")
+					(reference "FID2")
 					(unit 1)
 				)
@@
 		(in_pos_files yes)
 		(dnp no)
-		(property "Reference" "FID6"
+		(property "Reference" "FID4"
 			(at 35.179 19.1516 0)
 			(show_name no)
@@
 			(project "STS1_EEE"
 				(path "/81e05c2b-9a2c-430f-84ee-6a59968cd49a"
-					(reference "FID6")
+					(reference "FID4")
 					(unit 1)
 				)
@@
 		(in_pos_files yes)
 		(dnp no)
-		(property "Reference" "FID7"
+		(property "Reference" "FID6"
 			(at 50.419 19.1516 0)
 			(show_name no)
@@
 			(project "STS1_EEE"
 				(path "/81e05c2b-9a2c-430f-84ee-6a59968cd49a"
-					(reference "FID7")
+					(reference "FID6")
 					(unit 1)
 				)
@@
 		(in_pos_files yes)
 		(dnp no)
-		(property "Reference" "U10"
+		(property "Reference" "U2"
 			(at 132.7912 17.2466 0)
 			(show_name no)
@@
 			(project "STS1_EEE"
 				(path "/81e05c2b-9a2c-430f-84ee-6a59968cd49a"
-					(reference "U10")
-					(unit 1)
-				)
+					(reference "U2")
+					(unit 1)
+				)

Commit message: Fix ERC errors
Other:
- sheet STS1_connector ports: added none; removed COBC_SPI_[1..6], EDU_BOOT, EDU_EN, EDU_Heartbeat, EDU_SPI_[1..6], EDU_UPDATE, EPS_ANT_DEPLOYED, EPS_BAT_GOOD, EPS_CHARGING, UART_COBC_EDU_[1..2], UCI_COBC_3V3, UCI_COBC_UART_[1..2]
Changed lines of the file:
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@@
-			)
-		)
-		(pin "EDU_Heartbeat" input
-			(at 43.18 45.72 0)
-			(effects
-				(font
-					(size 1.27 1.27)
-				)
-				(justify right)
-			)
-		)
-		(pin "EDU_EN" input
-			(at 43.18 43.18 0)
-			(effects
-				(font
-					(size 1.27 1.27)
-				)
-				(justify right)
-			)
-		)
-		(pin "EDU_UPDATE" input
-			(at 43.18 48.26 0)
-			(effects
-				(font
-					(size 1.27 1.27)
-				)
-				(justify right)
-			)
-		)
-		(pin "EDU_SPI_[1..6]" input
-			(at 43.18 64.77 0)
-			(effects
-				(font
-					(size 1.27 1.27)
-				)
-				(justify right)
-			)
-		)
-		(pin "EPS_CHARGING" input
-			(at 43.18 52.07 0)
-			(effects
-				(font
-					(size 1.27 1.27)
-				)
-				(justify right)
-			)
-		)
-		(pin "EPS_ANT_DEPLOYED" input
-			(at 43.18 54.61 0)
-			(effects
-				(font
-					(size 1.27 1.27)
-				)
-				(justify right)
-			)
-		)
-		(pin "EPS_BAT_GOOD" input
-			(at 43.18 57.15 0)
-			(effects
-				(font
-					(size 1.27 1.27)
-				)
-				(justify right)
-			)
-		)
-		(pin "UCI_COBC_3V3" input
-			(at 43.18 60.96 0)
-			(effects
-				(font
-					(size 1.27 1.27)
-				)
-				(justify right)
-			)
-		)
-		(pin "UCI_COBC_UART_[1..2]" input
-			(at 43.18 72.39 0)
-			(effects
-				(font
-					(size 1.27 1.27)
-				)
-				(justify right)
-			)
-		)
-		(pin "COBC_SPI_[1..6]" input
-			(at 43.18 67.31 0)
-			(effects
-				(font
-					(size 1.27 1.27)
-				)
-				(justify right)
-			)
-		)
-		(pin "UART_COBC_EDU_[1..2]" input
-			(at 43.18 69.85 0)
-			(effects
-				(font
-					(size 1.27 1.27)
-				)
-				(justify right)
-			)
-		)
-		(pin "EDU_BOOT" input
-			(at 43.18 40.64 0)
-			(effects
-				(font
-					(size 1.27 1.27)
-				)
-				(justify right)
 			)
 		)
